File: sistemasolar.kicad_pcb (KiCad board)
At the start: 2 copper layers, 25 parts, among them J1 BATERIAS, J2 PANELSOLAR, J3 CONTROLVCC, Q1 2N3904, Q2 IRF9540N, Q3 2N3904, Q4 IRF9540N, Q5 IRF9540N, Q6 2N3904, Q7 2N3904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

Commit message: AgroneckPower finalizado
Parts:
- added ?: , , F.Cu at (125.2, 67.0)
- added ?: , , F.Cu at (114.5, 67.0)
- added F1: Fuse, Fuse:Fuseholder_Clip-5x20mm_Littelfuse_445-030_Inline_P20.50x5.20mm_D1.30mm_Horizontal, F.Cu at (55.4, 122.9)
- moved J3 34.4 mm to (102.2, 135.0)
- moved J1 20.5 mm to (143.0, 51.0), turned to -90 degrees
- moved R1 10.7 mm to (128.2, 121.9)
- moved R3 10.6 mm to (132.2, 121.8)
- moved U2 10.0 mm to (133.5, 83.8)
- moved D3 10.0 mm to (85.5, 123.1)
- moved U1 10.0 mm to (113.0, 84.0)
- moved D4 10.0 mm to (113.0, 123.1)
- moved Q1 10.0 mm to (123.2, 116.1)
- moved Q2 10.0 mm to (121.5, 108.1)
- moved Q3 10.0 mm to (137.5, 116.1)
- moved Q4 10.0 mm to (136.5, 108.1)
- moved Q5 10.0 mm to (92.0, 108.1)
- moved Q6 10.0 mm to (91.0, 116.8)
- moved Q7 10.0 mm to (107.9, 116.8)
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Connections:
- U4 pad 3: SUOUT+ -> Net-(U4-VOUT+)
Routing:
- net GND: track 371.0 -> 450.5 mm
- net Net-(U4-VOUT+): track 0.00 -> 31.0 mm
- net CONTROL2: track 72.2 -> 42.9 mm
- net CONTROL1: track 58.8 -> 31.4 mm
- net Net-(J1-Pin_1): track 17.8 -> 42.8 mm
- net Net-(J1-Pin_2): track 15.2 -> 34.0 mm
- net Net-(Q2-S): track 174.2 -> 190.6 mm
- net Net-(J1-Pin_4): track 39.4 -> 29.9 mm
- net SUOUT+: track 29.3 -> 20.0 mm
- net Net-(D3-K): track 165.9 -> 173.8 mm
- net CONTROL4: track 45.4 -> 40.7 mm
- net Net-(Q4-D): track 24.6 -> 20.8 mm
- net Net-(J2-Pin_1): track 47.6 -> 44.6 mm
- net Net-(Q2-D): track 24.2 -> 22.4 mm
- net Net-(Q7-C): track 12.8 -> 11.2 mm
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- added copper zone on B.Cu, net GND
Other:
- board text added: "AgroNomad"
- board text added: "SOLARIA"
