File: sistemasolar.kicad_sch (KiCad schematic)
At the start: 25 parts, among them J1 BATERIAS, J2 PANELSOLAR, J3 CONTROLVCC, Q1 2N3904, Q2 IRF9540N, Q3 2N3904, Q4 IRF9540N, Q5 IRF9540N, Q6 2N3904, Q7 2N3904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

Commit message: AgroneckPower finalizado
Parts:
- added F1: Fuse, Fuse:Fuseholder_Clip-5x20mm_Littelfuse_445-030_Inline_P20.50x5.20mm_D1.30mm_Horizontal, symbol Device:Fuse
Connections:
- net SUOUT+: now also F1.2; no longer U4.3 (VOUT+)
- new net: F1.1, U4.3 (VOUT+)
Changed lines of the file:
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@@
 	(wire
 		(pts
-			(xy 168.91 142.24) (xy 166.37 142.24)
+			(xy 166.37 142.24) (xy 170.18 142.24)
 		)
 		(stroke
@@
 		(pts
 			(xy 143.51 149.86) (xy 143.51 151.13)
+		)
+		(stroke
+			(width 0)
+			(type default)
+		)
+	)
+	(wire
+		(pts
+			(xy 177.8 142.24) (xy 181.61 142.24)
 		)
 		(stroke
@@
 	(global_label "SUOUT+"
 		(shape input)
-		(at 168.91 142.24 0)
+		(at 181.61 142.24 0)
 		(fields_autoplaced yes)
 		(effects
@@
 		)
 		(property "Intersheetrefs" "${INTERSHEET_REFS}"
-			(at 179.6362 142.24 0)
+			(at 192.3362 142.24 0)
 			(hide yes)
 			(show_name no)
@@
 					(unit 1)
 				)
+			)
+		)
+	)
+	(symbol
+		(lib_id "Device:Fuse")
+		(at 173.99 142.24 90)
+		(unit 1)
+		(body_style 1)
+		(exclude_from_sim no)
+		(in_bom yes)
+		(on_board yes)
+		(in_pos_files yes)
+		(dnp no)
+		(fields_autoplaced yes)
+		(property "Reference" "F1"
+			(at 173.99 135.89 90)
+			(show_name no)
+			(do_not_autoplace no)
+			(effects
+				(font
+					(size 1.27 1.27)
+				)
+			)
+		)
+		(property "Value" "Fuse"
+			(at 173.99 138.43 90)
+			(show_name no)
+			(do_not_autoplace no)
+			(effects
+				(font
+					(size 1.27 1.27)
+				)
+			)
+		)
+		(property "Footprint" "Fuse:Fuseholder_Clip-5x20mm_Littelfuse_445-030_Inline_P20.50x5.20mm_D1.30mm_Horizontal"
+			(at 173.99 144.018 90)
+			(hide yes)
+			(show_name no)
+			(do_not_autoplace no)
+			(effects
+				(font
+					(size 1.27 1.27)
+				)
+			)
+		)
+		(property "Datasheet" ""
+			(at 173.99 142.24 0)
+			(hide yes)
+			(show_name no)
+			(do_not_autoplace no)
+			(effects
+				(font
+					(size 1.27 1.27)
+				)
+			)
+		)
+		(property "Description" "Fuse"
+			(at 173.99 142.24 0)
+			(hide yes)
+			(show_name no)
+			(do_not_autoplace no)
+			(effects
+				(font
+					(size 1.27 1.27)
+				)
+			)
+		)
+		(pin "2"
+		)
+		(pin "1"
+		)
+		(instances
+			(project "sistemasolar"
+				(path "/37605b2f-a95c-4385-8c81-ccd587e35e25"
+					(reference "F1")
+					(unit 1)
+				)
